File: EagleSketches/Server/Server/Server wire chart.sch (EAGLE design)
At the start: 4 parts

Commit message: eglage
Elage
Parts:
- removed U$2: GY-BPM280, GY-BMP280:GY-BPM280
- added CAPACITOR: 47nF, capacitor-wima:C2,5-3
- added MQ135/FC22: (no value), RHT03_DHT-22_AM2302:MQ
Connections:
- removed net 3.3V: U$2.VCC
- new net N$1: MQ135/FC22.AD, U$1.IO4
- net 5V: now also MQ135/FC22.VCC
- net GND: now also MQ135/FC22.GND; no longer U$2.GND
- net N$2: now also U$1.IO14; no longer U$1.IO34
- net N$3: now also CAPACITOR.1, U$1.EN; no longer U$1.IO22, U$2.SCK
- net N$4: now also CAPACITOR.2, U$1.GND@32; no longer U$1.IO21, U$2.SDI
Changed lines of the file:
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@@
 <part name="AM2302" library="RHT03_DHT-22_AM2302" deviceset="RHT03_DHT-22_AM2302" device=""/>
 <part name="R1" library="SparkFun-Resistors" deviceset="10KOHM" device="-0402-1/16W-1%" value="10k"/>
-<part name="U$2" library="GY-BMP280" deviceset="GY-BPM280" device=""/>
+<part name="MQ135/FC22" library="RHT03_DHT-22_AM2302" deviceset="MQ" device=""/>
+<part name="CAPACITOR" library="capacitor-wima" library_urn="urn:adsk.eagle:library:116" deviceset="C" device="2,5-3" package3d_urn="urn:adsk.eagle:package:5436/1" value="47nF"/>
 </parts>
 <sheets>
@@
 <attribute name="VALUE" x="-3.556" y="60.96" size="1.778" layer="96" font="vector" rot="R90" align="top-center"/>
 </instance>
-<instance part="U$2" gate="G$1" x="106.68" y="106.68" smashed="yes" rot="R270"/>
+<instance part="MQ135/FC22" gate="G$1" x="96.52" y="66.04" smashed="yes">
+<attribute name="NAME" x="91.44" y="77.47" size="1.27" layer="94"/>
+<attribute name="VALUE" x="91.44" y="53.34" size="1.27" layer="94"/>
+</instance>
+<instance part="CAPACITOR" gate="G$1" x="38.1" y="93.98" smashed="yes" rot="R90">
+<attribute name="NAME" x="37.719" y="95.504" size="1.778" layer="95" rot="R180"/>
+<attribute name="VALUE" x="42.799" y="95.504" size="1.778" layer="96"/>
+</instance>
 </instances>
 <busses>
@@
 </segment>
 <segment>
-<pinref part="U$2" gate="G$1" pin="GND"/>
-<wire x1="91.44" y1="114.3" x2="86.36" y2="114.3" width="0.1524" layer="91"/>
-<label x="83.82" y="114.3" size="1.778" layer="95"/>
+<pinref part="MQ135/FC22" gate="G$1" pin="GND"/>
+<wire x1="86.36" y1="68.58" x2="78.74" y2="68.58" width="0.1524" layer="91"/>
+<label x="78.74" y="68.58" size="1.778" layer="95"/>
 </segment>
 </net>
@@
 <label x="0" y="55.88" size="1.778" layer="95"/>
 </segment>
+<segment>
+<pinref part="MQ135/FC22" gate="G$1" pin="VCC"/>
+<wire x1="86.36" y1="73.66" x2="78.74" y2="73.66" width="0.1524" layer="91"/>
+<label x="78.74" y="73.66" size="1.778" layer="95"/>
+</segment>
 </net>
 <net name="N$2" class="0">
@@
 <pinref part="R1" gate="G$1" pin="2"/>
 <wire x1="-15.24" y1="66.04" x2="-5.08" y2="66.04" width="0.1524" layer="91"/>
-<wire x1="-5.08" y1="66.04" x2="2.54" y2="66.04" width="0.1524" layer="91"/>
+<wire x1="-5.08" y1="66.04" x2="7.62" y2="66.04" width="0.1524" layer="91"/>
 <junction x="-5.08" y="66.04"/>
-<pinref part="U$1" gate="G$1" pin="IO34"/>
-<wire x1="2.54" y1="66.04" x2="2.54" y2="73.66" width="0.1524" layer="91"/>
-<wire x1="2.54" y1="73.66" x2="20.32" y2="73.66" width="0.1524" layer="91"/>
+<pinref part="U$1" gate="G$1" pin="IO14"/>
+<wire x1="20.32" y1="55.88" x2="7.62" y2="55.88" width="0.1524" layer="91"/>
+<wire x1="7.62" y1="55.88" x2="7.62" y2="66.04" width="0.1524" layer="91"/>
 </segment>
 </net>
-<net name="3.3V" class="0">
+<net name="N$1" class="0">
 <segment>
-<pinref part="U$2" gate="G$1" pin="VCC"/>
-<wire x1="91.44" y1="119.38" x2="83.82" y2="119.38" width="0.1524" layer="91"/>
-<label x="83.82" y="119.38" size="1.778" layer="95"/>
+<pinref part="U$1" gate="G$1" pin="IO4"/>
+<wire x1="55.88" y1="53.34" x2="63.5" y2="53.34" width="0.1524" layer="91"/>
+<wire x1="63.5" y1="53.34" x2="63.5" y2="58.42" width="0.1524" layer="91"/>
+<pinref part="MQ135/FC22" gate="G$1" pin="AD"/>
+<wire x1="63.5" y1="58.42" x2="86.36" y2="58.42" width="0.1524" layer="91"/>
+</segment>
+</net>
+<net name="N$3" class="0">
+<segment>
+<pinref part="U$1" gate="G$1" pin="EN"/>
+<wire x1="20.32" y1="81.28" x2="12.7" y2="81.28" width="0.1524" layer="91"/>
+<wire x1="12.7" y1="81.28" x2="12.7" y2="93.98" width="0.1524" layer="91"/>
+<pinref part="CAPACITOR" gate="G$1" pin="1"/>
+<wire x1="12.7" y1="93.98" x2="35.56" y2="93.98" width="0.1524" layer="91"/>
 </segment>
 </net>
 <net name="N$4" class="0">
 <segment>
-<pinref part="U$2" gate="G$1" pin="SDI"/>
-<wire x1="91.44" y1="104.14" x2="63.5" y2="104.14" width="0.1524" layer="91"/>
-<wire x1="63.5" y1="104.14" x2="63.5" y2="71.12" width="0.1524" layer="91"/>
-<pinref part="U$1" gate="G$1" pin="IO21"/>
-<wire x1="63.5" y1="71.12" x2="55.88" y2="71.12" width="0.1524" layer="91"/>
-</segment>
-</net>
-<net name="N$3" class="0">
-<segment>
-<pinref part="U$2" gate="G$1" pin="SCK"/>
-<wire x1="91.44" y1="109.22" x2="91.44" y2="106.68" width="0.1524" layer="91"/>
-<wire x1="91.44" y1="106.68" x2="60.96" y2="106.68" width="0.1524" layer="91"/>
-<pinref part="U$1" gate="G$1" pin="IO22"/>
-<wire x1="60.96" y1="106.68" x2="60.96" y2="78.74" width="0.1524" layer="91"/>
-<wire x1="60.96" y1="78.74" x2="55.88" y2="78.74" width="0.1524" layer="91"/>
+<pinref part="U$1" gate="G$1" pin="GND@32"/>
+<wire x1="55.88" y1="68.58" x2="73.66" y2="68.58" width="0.1524" layer="91"/>
+<wire x1="73.66" y1="68.58" x2="73.66" y2="93.98" width="0.1524" layer="91"/>
+<pinref part="CAPACITOR" gate="G$1" pin="2"/>
+<wire x1="73.66" y1="93.98" x2="43.18" y2="93.98" width="0.1524" layer="91"/>
 </segment>
 </net>
@@
 </drawing>
 <compatibility>
+<note version="8.2" severity="warning">
+Since Version 8.2, EAGLE supports online libraries. The ids
+of those online libraries will not be understood (or retained)
+with this version.
+</note>
 <note version="8.3" severity="warning">
 Since Version 8.3, EAGLE supports URNs for individual library
@@
 will not be understood (or retained) with this version.
 </note>
+<note version="8.3" severity="warning">
+Since Version 8.3, EAGLE supports the association of 3D packages
+with devices in libraries, schematics, and board files. Those 3D
+packages will not be understood (or retained) with this version.
+</note>
 </compatibility>
