File: EagleSketches/Client/main.brd (EAGLE design)
At the start: 100 x 80 mm, 22 parts, among them J1 MICRO-SD-PUSH-PUSH-EXT-PIN, U1 LM386N

Commit message: Working audio
Parts:
- added C3: 0.1uF, SparkFun-Capacitors:CAP-PTH-SMALL-KIT
Connections:
- new net N$30: C3.2, U1.3
- net N$23: now also C3.1; no longer U1.3
Changed lines of the file:
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@@
 <attribute name="VALUE" x="-144.78" y="-52.07" size="0.5" layer="27" align="center"/>
+</element>
+<element name="C3" library="SparkFun-Capacitors" package="CAP-PTH-SMALL-KIT" value="0.1uF" x="-149.86" y="-64.77" smashed="yes">
+<attribute name="PROD_ID" value="CAP-08370" x="-149.86" y="-64.77" size="1.778" layer="27" display="off"/>
 </element>
 </elements>
@@
 <contactref element="R7" pad="P$2"/>
 </signal>
-<signal name="N$23">
-<contactref element="VR2" pad="1"/>
-<contactref element="U1" pad="3"/>
-<wire x1="-127" y1="-16.51" x2="-126.44" y2="-23.4" width="0" layer="19" extent="1-1"/>
-</signal>
 <signal name="N$21">
 <contactref element="VR2" pad="2A"/>
@@
 <wire x1="-43.19" y1="88.7" x2="-149.13" y2="-41.57" width="0" layer="19" extent="1-1"/>
 </signal>
+<signal name="N$23">
+<contactref element="VR2" pad="1"/>
+<contactref element="C3" pad="1"/>
+<wire x1="-126.44" y1="-23.4" x2="-151.257" y2="-64.77" width="0" layer="19" extent="1-1"/>
+</signal>
+<signal name="N$30">
+<contactref element="C3" pad="2"/>
+<contactref element="U1" pad="3"/>
+<wire x1="-127" y1="-16.51" x2="-148.463" y2="-64.77" width="0" layer="19" extent="1-1"/>
+</signal>
 </signals>

Commit message: Endelige versioner af koden
Parts:
- added BT2: (no value), SparkFun-Batteries:BATTCON_9V
- added C4: 47nF, SparkFun-Capacitors:0603
- added S1, S7: (no value), switch:MS243
Connections:
- new net N$31: S1.2, U1.6
- new net N$32: C4.2, U$2.1
- new net N$33: BT2.-, S7.1
- net 5V: now also S7.2
- net GND: now also BT2.+, C4.1
- net N$22: now also S1.1; no longer U1.6
Changed lines of the file:
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@@
 <attribute name="PROD_ID" value="CAP-08370" x="-149.86" y="-64.77" size="1.778" layer="27" display="off"/>
+</element>
+<element name="S1" library="switch" library_urn="urn:adsk.eagle:library:380" package="MS243" package3d_urn="urn:adsk.eagle:package:27683/1" value="" x="-148.59" y="-72.39" smashed="yes">
+<attribute name="NAME" x="-144.145" y="-73.66" size="1.778" layer="25" ratio="10"/>
+<attribute name="POPULARITY" value="3" x="-148.59" y="-72.39" size="1.778" layer="27" display="off"/>
+<attribute name="VALUE" x="-144.145" y="-76.2" size="1.778" layer="27" ratio="10"/>
+</element>
+<element name="BT2" library="SparkFun-Batteries" package="BATTCON_9V" value="" x="-97.79" y="-87.63" smashed="yes">
+<attribute name="NAME" x="-151.13" y="-93.98" size="0.6096" layer="25" font="vector" ratio="20" rot="R90" align="bottom-center"/>
+<attribute name="PROD_ID" value="BATT-10855" x="-97.79" y="-87.63" size="1.778" layer="27" display="off"/>
+<attribute name="VALUE" x="-123.19" y="-93.98" size="0.6096" layer="27" font="vector" ratio="20" rot="R90" align="top-center"/>
+</element>
+<element name="S7" library="switch" library_urn="urn:adsk.eagle:library:380" package="MS243" package3d_urn="urn:adsk.eagle:package:27683/1" value="" x="-148.59" y="-115.57" smashed="yes">
+<attribute name="NAME" x="-144.145" y="-116.84" size="1.778" layer="25" ratio="10"/>
+<attribute name="POPULARITY" value="3" x="-148.59" y="-115.57" size="1.778" layer="27" display="off"/>
+<attribute name="VALUE" x="-144.145" y="-119.38" size="1.778" layer="27" ratio="10"/>
+</element>
+<element name="C4" library="SparkFun-Capacitors" package="0603" value="47nF" x="-151.13" y="-123.19" smashed="yes">
+<attribute name="NAME" x="-151.13" y="-122.428" size="0.6096" layer="25" font="vector" ratio="20" align="bottom-center"/>
+<attribute name="PROD_ID" value="CAP-08605" x="-151.13" y="-123.19" size="1.778" layer="27" display="off"/>
+<attribute name="VALUE" x="-151.13" y="-123.952" size="0.6096" layer="27" font="vector" ratio="20" align="top-center"/>
 </element>
 </elements>
@@
 <contactref element="J1" pad="11"/>
 <contactref element="J1" pad="12"/>
+<contactref element="BT2" pad="+"/>
+<contactref element="C4" pad="1"/>
 <wire x1="-152.53" y1="-42.17" x2="-152.53" y2="-51.67" width="0" layer="19" extent="1-1"/>
 <wire x1="-148.03" y1="-41.57" x2="-152.53" y2="-42.17" width="0" layer="19" extent="1-1"/>
@@
 <wire x1="-81.28" y1="-40.64" x2="-124.46" y2="-16.51" width="0" layer="19" extent="1-1"/>
 <wire x1="-56.44" y1="-23.4" x2="-81.28" y2="-40.64" width="0" layer="19" extent="1-1"/>
+<wire x1="-97.79" y1="-87.63" x2="-81.28" y2="-40.64" width="0" layer="19" extent="1-1"/>
 <wire x1="-101.76" y1="58.77" x2="-121.666" y2="6.35" width="0" layer="19" extent="1-1"/>
 <wire x1="-91.6" y1="58.77" x2="-101.76" y2="58.77" width="0" layer="19" extent="1-1"/>
@@
 <wire x1="-99.06" y1="110.49" x2="-88.9" y2="110.49" width="0" layer="19" extent="1-1"/>
 <wire x1="-22.15" y1="102.33" x2="-58.42" y2="110.49" width="0" layer="19" extent="1-1"/>
+<wire x1="-151.98" y1="-123.19" x2="-97.79" y2="-87.63" width="0" layer="19" extent="1-1"/>
 </signal>
 <signal name="5V">
@@
 <contactref element="U$2" pad="19"/>
 <contactref element="J1" pad="4"/>
+<contactref element="S7" pad="2"/>
+<wire x1="-148.59" y1="-114.2238" x2="-145.83" y2="-41.57" width="0" layer="19" extent="1-1"/>
 <wire x1="-99.22" y1="58.77" x2="-145.83" y2="-41.57" width="0" layer="19" extent="1-1"/>
 <wire x1="-97.15" y1="97.33" x2="-99.22" y2="58.77" width="0" layer="19" extent="1-1"/>
@@
 <wire x1="-40.65" y1="66.05" x2="-131.44" y2="-28.4" width="0" layer="19" extent="1-1"/>
 </signal>
-<signal name="N$22">
-<contactref element="BT1" pad="-"/>
-<contactref element="U1" pad="6"/>
-<wire x1="-127" y1="-8.89" x2="-81.28" y2="-53.594" width="0" layer="19" extent="1-1"/>
-</signal>
 <signal name="N$5">
 <contactref element="U$2" pad="24"/>
@@
 <wire x1="-127" y1="-16.51" x2="-148.463" y2="-64.77" width="0" layer="19" extent="1-1"/>
 </signal>
+<signal name="N$22">
+<contactref element="BT1" pad="-"/>
+<contactref element="S1" pad="1"/>
+<wire x1="-81.28" y1="-53.594" x2="-148.59" y2="-73.7362" width="0" layer="19" extent="1-1"/>
+</signal>
+<signal name="N$31">
+<contactref element="S1" pad="2"/>
+<contactref element="U1" pad="6"/>
+<wire x1="-127" y1="-8.89" x2="-148.59" y2="-71.0438" width="0" layer="19" extent="1-1"/>
+</signal>
+<signal name="N$33">
+<contactref element="BT2" pad="-"/>
+<contactref element="S7" pad="1"/>
+<wire x1="-148.59" y1="-116.9162" x2="-97.79" y2="-100.584" width="0" layer="19" extent="1-1"/>
+</signal>
+<signal name="N$32">
+<contactref element="U$2" pad="1"/>
+<contactref element="C4" pad="2"/>
+<wire x1="-60.97" y1="66.05" x2="-150.28" y2="-123.19" width="0" layer="19" extent="1-1"/>
+</signal>
 </signals>
