File: EagleSketches/Client/main.sch (EAGLE design)
At the start: 23 parts, among them J1 MICRO-SD-PUSH-PUSH-EXT-PIN, U1 LM386N

Commit message: Endelige versioner af koden
Parts:
- added BT2: (no value), SparkFun-Batteries:BATTERY-9V
- added C4: 47nF, SparkFun-Capacitors:47NF-0603-25V-5%
- added S1, S7: (no value), switch:MS243
Connections:
- new net N$31: S1.S, U1.V+
- new net N$32: C4.2, U$2.3V3
- new net N$33: BT2.-, S7.P
- net 5V: now also S7.S
- net GND: now also BT2.+, C4.1
- net N$22: now also S1.P; no longer U1.V+
Changed lines of the file:
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@@
 <part name="J1" library="SparkFun-Connectors" deviceset="MICRO-SD" device="-PUSH-PUSH-EXT-PIN"/>
 <part name="C3" library="SparkFun-Capacitors" deviceset="0.1UF" device="-KIT-EZ-50V-20%" value="0.1uF"/>
+<part name="S1" library="switch" library_urn="urn:adsk.eagle:library:380" deviceset="MS243" device="" package3d_urn="urn:adsk.eagle:package:27683/1"/>
+<part name="BT2" library="SparkFun-Batteries" deviceset="BATTERY" device="-9V"/>
+<part name="S7" library="switch" library_urn="urn:adsk.eagle:library:380" deviceset="MS243" device="" package3d_urn="urn:adsk.eagle:package:27683/1"/>
+<part name="C4" library="SparkFun-Capacitors" deviceset="47NF" device="-0603-25V-5%" value="47nF"/>
 </parts>
 <sheets>
@@
 <attribute name="VALUE" x="-30.861" y="113.284" size="1.778" layer="96" font="vector" rot="R90"/>
 </instance>
+<instance part="S1" gate="1" x="-30.48" y="137.16" smashed="yes" rot="R270">
+<attribute name="NAME" x="-27.305" y="140.97" size="1.778" layer="95"/>
+<attribute name="VALUE" x="-27.305" y="138.43" size="1.778" layer="96"/>
+</instance>
+<instance part="BT2" gate="G$1" x="12.7" y="22.86" smashed="yes">
+<attribute name="NAME" x="12.7" y="27.178" size="1.778" layer="95" font="vector" align="bottom-center"/>
+<attribute name="VALUE" x="12.7" y="18.542" size="1.778" layer="96" font="vector" align="top-center"/>
+</instance>
+<instance part="S7" gate="1" x="27.94" y="25.4" smashed="yes" rot="R270">
+<attribute name="NAME" x="31.115" y="29.21" size="1.778" layer="95"/>
+<attribute name="VALUE" x="31.115" y="26.67" size="1.778" layer="96"/>
+</instance>
+<instance part="C4" gate="G$1" x="15.24" y="88.9" smashed="yes">
+<attribute name="NAME" x="16.764" y="91.821" size="1.778" layer="95" font="vector"/>
+<attribute name="VALUE" x="16.764" y="86.741" size="1.778" layer="96" font="vector"/>
+</instance>
 </instances>
 <busses>
@@
 <label x="-73.66" y="88.9" size="1.778" layer="95"/>
 </segment>
+<segment>
+<pinref part="BT2" gate="G$1" pin="+"/>
+<wire x1="7.62" y1="22.86" x2="5.08" y2="22.86" width="0.1524" layer="91"/>
+<label x="2.54" y="22.86" size="1.778" layer="95"/>
+</segment>
+<segment>
+<pinref part="C4" gate="G$1" pin="1"/>
+<wire x1="15.24" y1="93.98" x2="20.32" y2="93.98" width="0.1524" layer="91"/>
+<label x="20.32" y="93.98" size="1.778" layer="95"/>
+</segment>
 </net>
 <net name="5V" class="0">
@@
 <wire x1="-76.2" y1="109.22" x2="-71.12" y2="109.22" width="0.1524" layer="91"/>
 <label x="-73.66" y="109.22" size="1.778" layer="95"/>
+</segment>
+<segment>
+<pinref part="S7" gate="1" pin="S"/>
+<wire x1="33.02" y1="22.86" x2="35.56" y2="22.86" width="0.1524" layer="91"/>
+<label x="35.56" y="22.86" size="1.778" layer="95"/>
 </segment>
 </net>
@@
 </segment>
 </net>
-<net name="N$22" class="0">
-<segment>
-<pinref part="BT1" gate="G$1" pin="-"/>
-<wire x1="-38.1" y1="134.62" x2="-22.86" y2="134.62" width="0.1524" layer="91"/>
-<pinref part="U1" gate="G1" pin="V+"/>
-<wire x1="-22.86" y1="134.62" x2="-22.86" y2="121.92" width="0.1524" layer="91"/>
-</segment>
-</net>
 <net name="N$5" class="0">
 <segment>
@@
 </segment>
 </net>
+<net name="N$22" class="0">
+<segment>
+<pinref part="BT1" gate="G$1" pin="-"/>
+<pinref part="S1" gate="1" pin="P"/>
+<wire x1="-38.1" y1="134.62" x2="-35.56" y2="134.62" width="0.1524" layer="91"/>
+</segment>
+</net>
+<net name="N$31" class="0">
+<segment>
+<pinref part="S1" gate="1" pin="S"/>
+<pinref part="U1" gate="G1" pin="V+"/>
+<wire x1="-25.4" y1="134.62" x2="-22.86" y2="134.62" width="0.1524" layer="91"/>
+<wire x1="-22.86" y1="134.62" x2="-22.86" y2="121.92" width="0.1524" layer="91"/>
+</segment>
+</net>
+<net name="N$33" class="0">
+<segment>
+<pinref part="BT2" gate="G$1" pin="-"/>
+<pinref part="S7" gate="1" pin="P"/>
+<wire x1="17.78" y1="22.86" x2="22.86" y2="22.86" width="0.1524" layer="91"/>
+</segment>
+</net>
+<net name="N$32" class="0">
+<segment>
+<pinref part="U$2" gate="G$1" pin="3V3"/>
+<pinref part="C4" gate="G$1" pin="2"/>
+<wire x1="7.62" y1="86.36" x2="15.24" y2="86.36" width="0.1524" layer="91"/>
+</segment>
+</net>
